Commit message: Add YAML-driven PS4 teleop for Edge Servo, gripper, and named poses.
Introduce ps4_mapper with configurable mappings, edge_teleop_sim launch, L7 jaw mesh fix, and sim_executor t=0 sampling for gripper trajectories.

Co-authored-by: Cursor <cursoragent@cursor.com>

File: src/a3_description/urdf/el_a3.urdf (robot description, URDF)
Before this commit: robot EL-A3, 10 links, 9 joints
Links:
- added link gripper_palm_link, mass 0.02; collision box size=0.028 0.012 0.018; visual box size=0.028 0.012 0.018
- added link left_finger_link, mass 0.015; collision box size=0.010 0.014 0.038; visual box size=0.010 0.014 0.038
- added link right_finger_link, mass 0.015; collision box size=0.010 0.014 0.038; visual box size=0.010 0.014 0.038
- link gripper_link: mass 0.05 -> 0.01
- link l5_l6_urdf_asm: geometry collision mesh filename=package://a3_description/meshes/el05_l6.stl; visual mesh filename=package://a3_description/meshes/el05_l6.stl
Joints:
- added joint gripper_palm_joint: type fixed, parent l5_l6_urdf_asm, child gripper_palm_link, origin xyz=0 0 0 rpy=0 0 0
- added joint left_finger_joint: type prismatic, parent l5_l6_urdf_asm, child left_finger_link, origin xyz=0 0.022 0 rpy=0 0 0, axis 0 -1 0, limit lower=0 upper=0.022 effort=20 velocity=0.05, mimic joint=L7_joint multiplier=0.01401 offset=0
- added joint right_finger_joint: type prismatic, parent l5_l6_urdf_asm, child right_finger_link, origin xyz=0 -0.022 0 rpy=0 0 0, axis 0 1 0, limit lower=0 upper=0.022 effort=20 velocity=0.05, mimic joint=L7_joint multiplier=0.01401 offset=0
- joint L7_joint: limit lower=-1.5708 upper=1.5708 effort=6.0 velocity=50 -> lower=0 upper=1.5708 effort=6.0 velocity=50

File: src/a3_description/urdf/el_a3.urdf.xacro (robot description, xacro)
@@ -13,4 +13,5 @@
   <!-- Include ros2_control -->
   <xacro:include filename="$(find a3_description)/urdf/el_a3_ros2_control.xacro"/>
+  <xacro:include filename="$(find a3_description)/urdf/gripper_mimic.xacro"/>
   <!-- Materials -->
   <material name="orange">
@@ -181,18 +182,4 @@
       </geometry>
     </collision>
-    <!-- Part jaw -->
-    <visual>
-      <origin xyz="0 0 -0.0755" rpy="3.14159 0 0"/>
-      <geometry>
-        <mesh filename="package://a3_description/meshes/jaw.stl"/>
-      </geometry>
-      <material name="orange"/>
-    </visual>
-    <collision>
-      <origin xyz="0 0 -0.0755" rpy="3.14159 0 0"/>
-      <geometry>
-        <mesh filename="package://a3_description/meshes/jaw.stl"/>
-      </geometry>
-    </collision>
   </link>
   <!-- End Effector link -->
@@ -259,20 +246,6 @@
     <child link="end_effector"/>
   </joint>
-  <!-- Joint L7 (${wrist_motor_type} Motor 7 - Gripper, separate kinematic branch) -->
-  <joint name="L7_joint" type="revolute">
-    <origin xyz="0 0 -0.074" rpy="0 0 0"/>
-    <parent link="l5_l6_urdf_asm"/>
-    <child link="gripper_link"/>
-    <axis xyz="0 0 1"/>
-    <limit effort="${wrist_effort}" velocity="50" lower="-1.5708" upper="1.5708"/>
-    <dynamics damping="0.05" friction="0.05"/>
-  </joint>
-  <link name="gripper_link">
-    <inertial>
-      <mass value="0.05"/>
-      <origin xyz="0 0 0"/>
-      <inertia ixx="0.0001" ixy="0" ixz="0" iyy="0.0001" iyz="0" izz="0.0001"/>
-    </inertial>
-  </link>
+  <!-- Joint L7 + mimic parallel fingers (see gripper_mimic.xacro) -->
+  <xacro:el_a3_gripper parent_link="l5_l6_urdf_asm" wrist_effort="${wrist_effort}"/>
   <!-- ros2_control interface -->
   <xacro:el_a3_ros2_control

Commit message: Simplify L7 gripper URDF and harden PS4 teleop input handling.
Drop mimic-finger xacro for jaw mesh on L7, add sim_executor Servo streaming merge, and fix gripper polarity plus D-pad hysteresis and joy warmup.

Co-authored-by: Cursor <cursoragent@cursor.com>

File: src/a3_description/urdf/el_a3.urdf (robot description, URDF)
Before this commit: robot EL-A3, 13 links, 12 joints
Links:
- removed link gripper_palm_link
- removed link left_finger_link
- removed link right_finger_link
- link gripper_link: mass 0.01 -> 0.05; geometry collision mesh filename=package://a3_description/meshes/jaw.stl; visual mesh filename=package://a3_description/meshes/jaw.stl
Joints:
- removed joint gripper_palm_joint
- removed joint left_finger_joint
- removed joint right_finger_joint
- joint L7_joint: limit lower=0 upper=1.5708 effort=6.0 velocity=50 -> lower=-1.5708 upper=1.5708 effort=6.0 velocity=50

File: src/a3_description/urdf/el_a3.urdf.xacro (robot description, xacro)
@@ -13,5 +13,4 @@
   <!-- Include ros2_control -->
   <xacro:include filename="$(find a3_description)/urdf/el_a3_ros2_control.xacro"/>
-  <xacro:include filename="$(find a3_description)/urdf/gripper_mimic.xacro"/>
   <!-- Materials -->
   <material name="orange">
@@ -246,6 +245,33 @@
     <child link="end_effector"/>
   </joint>
-  <!-- Joint L7 + mimic parallel fingers (see gripper_mimic.xacro) -->
-  <xacro:el_a3_gripper parent_link="l5_l6_urdf_asm" wrist_effort="${wrist_effort}"/>
+  <!-- Joint L7 (${wrist_motor_type} Motor 7 - Gripper, separate kinematic branch) -->
+  <joint name="L7_joint" type="revolute">
+    <origin xyz="0 0 -0.074" rpy="0 0 0"/>
+    <parent link="l5_l6_urdf_asm"/>
+    <child link="gripper_link"/>
+    <axis xyz="0 0 1"/>
+    <limit effort="${wrist_effort}" velocity="50" lower="-1.5708" upper="1.5708"/>
+    <dynamics damping="0.05" friction="0.05"/>
+  </joint>
+  <link name="gripper_link">
+    <inertial>
+      <mass value="0.05"/>
+      <origin xyz="0 0 0"/>
+      <inertia ixx="0.0001" ixy="0" ixz="0" iyy="0.0001" iyz="0" izz="0.0001"/>
+    </inertial>
+    <visual>
+      <origin xyz="0 0 -0.0015" rpy="3.14159 0 0"/>
+      <geometry>
+        <mesh filename="package://a3_description/meshes/jaw.stl"/>
+      </geometry>
+      <material name="orange"/>
+    </visual>
+    <collision>
+      <origin xyz="0 0 -0.0015" rpy="3.14159 0 0"/>
+      <geometry>
+        <mesh filename="package://a3_description/meshes/jaw.stl"/>
+      </geometry>
+    </collision>
+  </link>
   <!-- ros2_control interface -->
   <xacro:el_a3_ros2_control

Commit message: Add F29-F34 motor debug downlink, gripper force fixes and recalibration
- F29: recover control_mode publishing defect from /a3/control_mode
- F30: gripper force timeout now honors command-provided timeout_s
- F31: gripper target_position telemetry, dual-curve panel, NaN telemetry sanitize
- F32: web motor debug page backend - CAN scan, MIT hold, motor state/scan
  collect services and msgs in a3_can_bridge, MQTT motor_* ops in bridge
- F33: gripper force fixes - contact travel gate from open stop, default
  grasp timeout 15s, release compliance (kp/kd/duration), zero-torque
  direct full-open, force-loop target position telemetry
- Recalibrate L7 zero at full-open stop, close = 1.7945 rad
- Add motor_debug_test.py and mqtt_force_ladder_test.py (F34 acceptance)
- Add LL-008..LL-015 lessons learned, CLAUDE.md

Co-Authored-By: Claude Code <noreply@anthropic.com>

File: src/a3_description/urdf/el_a3.urdf (robot description, URDF)
Before this commit: robot EL-A3, 10 links, 9 joints
Joints:
- joint L7_joint: axis 0 0 1 -> 0 0 -1; limit lower=-1.5708 upper=1.5708 effort=6.0 velocity=50 -> lower=0 upper=1.8 effort=6.0 velocity=50
