Commit message: F69: arm-specific servo singularity thresholds 25/50 + ready ridge point, regenerate stale URDF, sync F108 acceptance
Real-machine READY L1 jog made the whole arm go limp and sag under
gravity regardless of stick direction (LL-082). bag evidence showed
kp=80/kd=2 unchanged throughout: MoveIt Servo's singularity velocity
scaling (MoveIt defaults 17/30) tripped status 1/6 continuously,
shrinking twist to ~zero so the 20 ms target tracked feedback within
~0.003 rad and kp restoring torque (~0.24 Nm) lost to gravity
(~3.4 Nm). pinocchio full-arm Jacobian grid analysis showed this
non-spherical-wrist arm is inherently ill-conditioned (workspace
valley cond ~13.3, common region 13-25; SRDF ready cond=982 from a
locked elbow, SRDF home=23), so the default 17 sat inside the normal
workspace. Fix is joint point + threshold together:
- ready override -> [0,1.6,-0.7,0,0,0] valley/ridge point
  (cond 13.3, gravity torque ~2.4 Nm); pose data lives in
  ~/.a3/poses.yaml (F39 precedence), home/zero unchanged
- lower/hard_stop singularity thresholds 17/30 -> 25/50 in
  servo_config.yaml: <25 full speed, 25-50 scale, >=50 halt still
  ~2x before true singularities (cond >=100); re-calibration red
  line documented in SAFETY.md if future geometry shifts cond
- sim verified ROS_DOMAIN_ID=58: four independent 3 s twists from
  fresh ready, status 0 throughout, cond peaks 13.7-22.2 <25;
  real-hardware acceptance pending power-up

Also:
- regenerate stale generated el_a3.urdf from committed xacros
  (CRLF->LF; now reflects F98 L7 axis +Z and [0,1.78] calibrated
  limit, and F72/F107/F108 ros2_control hardware params: can0,
  pinocchio gravity feedforward, F49 inertia scales, position
  kp/kd, velocity/acceleration limits)
- F72/F73 vcan acceptance assertions follow F108 position-mode
  gravity feedforward now default-on: L1-L6 CAN torque_ff must
  match independent Python-pinocchio RNEA x direction (with F49
  fitted inertias loaded from inertia_params.yaml, tol 0.02 Nm),
  L7 torque_ff stays 0
- LL-082 new lesson; REQUIREMENTS F69 done(sim), SAFETY,
  QUICKSTART synced

File: src/a3_description/urdf/el_a3.urdf (robot description, URDF)
Before this commit: robot EL-A3, 10 links, 9 joints
Joints:
- joint L7_joint: axis 0 0 -1 -> 0 0 1; limit lower=0 upper=1.8 effort=6.0 velocity=50 -> lower=0.0 upper=1.78 effort=6.0 velocity=50
