Commit message: Add F72 real-motor SystemInterface plugin (SocketCAN + MIT) with vcan acceptance
New a3_hardware_interface package exports A3MITHardwareInterface so
controller_manager drives the 7 MIT motors directly over SocketCAN;
JTC/JSB/move_group wiring is unchanged from F70 and motor_protocol_node
is fully bypassed on this path. Verified on vcan0 with a 7-motor feedback
simulator: f72 acceptance ALL PASS (trajectory tracking, CAN mapping,
kp/kd, no legacy nodes). Real-hardware acceptance pending power-on.

Co-Authored-By: Claude Sonnet 4.6 <noreply@anthropic.com>

File: src/a3_description/urdf/el_a3.urdf.xacro (robot description, xacro)
@@ -5,4 +5,5 @@
   <!-- Arguments -->
   <xacro:arg name="use_mock_hardware" default="false"/>
+  <xacro:arg name="use_real_hardware" default="false"/>
   <xacro:arg name="can_interface" default="can0"/>
   <xacro:arg name="host_can_id" default="253"/>
@@ -277,4 +278,5 @@
   <xacro:el_a3_ros2_control
     use_mock_hardware="$(arg use_mock_hardware)"
+    use_real_hardware="$(arg use_real_hardware)"
     can_interface="$(arg can_interface)"
     host_can_id="$(arg host_can_id)"

File: src/a3_description/urdf/el_a3_ros2_control.xacro (robot description, xacro)
@@ -2,5 +2,5 @@
 <!-- EL-A3 ros2_control configuration -->
 <robot xmlns:xacro="http://www.ros.org/wiki/xacro">
-  <xacro:macro name="el_a3_ros2_control" params="use_mock_hardware can_interface host_can_id wrist_motor_type">
+  <xacro:macro name="el_a3_ros2_control" params="use_mock_hardware use_real_hardware can_interface host_can_id wrist_motor_type">
     <!-- Wrist motor effort limits based on motor type -->
     <xacro:property name="wrist_effort_max" value="${5.5 if wrist_motor_type == 'RS05' else 6.0}"/>
@@ -15,4 +15,13 @@
         </xacro:if>
         <xacro:unless value="${use_mock_hardware}">
+          <xacro:if value="${use_real_hardware}">
+            <!-- F72: real motors via ros2_control SystemInterface (SocketCAN + MIT).
+                 Per-joint motor_id/direction/position_offset read from joint params below. -->
+            <plugin>a3_hardware_interface/A3MITHardwareInterface</plugin>
+            <param name="can_interface">${can_interface}</param>
+            <param name="kp">80.0</param>
+            <param name="kd">2.0</param>
+          </xacro:if>
+          <xacro:unless value="${use_real_hardware}">
           <!-- Board runtime uses a3_can_bridge topic stack (not this plugin).
                Keep mock GenericSystem so MoveIt/demo can still load without el_a3_hardware. -->
@@ -75,4 +84,5 @@
           <param name="gravity_comp_L6_cos">0.0</param>
           <param name="gravity_comp_L6_offset">0.0</param>
+          </xacro:unless>
         </xacro:unless>
       </hardware>

Commit message: Add F85: velocity-adaptive free-drive Kd (Lorentzian + EMA), vcan acceptance 29/29
Ports the official EDULITE_A3 computeAdaptiveKd into the hardware plugin's
EFFORT CAN path: high damping at rest, low damping when pushed, EMA-smoothed.
Wires the six xacro params that were declared since 2026-08-21 but never
parsed (LL-088); per-joint kd_max overrides on L4-L7; false falls back to
fixed zero_torque_kd=0.3. RNEA gravity-comp controller unchanged.

Co-Authored-By: Claude Sonnet 4.6 <noreply@anthropic.com>

File: src/a3_description/urdf/el_a3.urdf.xacro (robot description, xacro)
@@ -9,4 +9,5 @@
   <xacro:arg name="host_can_id" default="253"/>
   <xacro:arg name="wrist_motor_type" default="EL05"/>
+  <xacro:arg name="adaptive_kd_enabled" default="true"/>
   <!-- Wrist motor parameters (EL05: 6Nm, RS05: 5.5Nm) -->
   <xacro:property name="wrist_motor_type" value="$(arg wrist_motor_type)"/>
@@ -281,4 +282,5 @@
     can_interface="$(arg can_interface)"
     host_can_id="$(arg host_can_id)"
-    wrist_motor_type="$(arg wrist_motor_type)"/>
+    wrist_motor_type="$(arg wrist_motor_type)"
+    adaptive_kd_enabled="$(arg adaptive_kd_enabled)"/>
 </robot>

File: src/a3_description/urdf/el_a3_ros2_control.xacro (robot description, xacro)
@@ -2,5 +2,5 @@
 <!-- EL-A3 ros2_control configuration -->
 <robot xmlns:xacro="http://www.ros.org/wiki/xacro">
-  <xacro:macro name="el_a3_ros2_control" params="use_mock_hardware use_real_hardware can_interface host_can_id wrist_motor_type">
+  <xacro:macro name="el_a3_ros2_control" params="use_mock_hardware use_real_hardware can_interface host_can_id wrist_motor_type adaptive_kd_enabled">
     <!-- Wrist motor effort limits based on motor type -->
     <xacro:property name="wrist_effort_max" value="${5.5 if wrist_motor_type == 'RS05' else 6.0}"/>
@@ -24,4 +24,12 @@
             <param name="temp_warn_c">90.0</param>
             <param name="temp_protect_c">95.0</param>
+            <!-- F85: velocity-adaptive free-drive damping (el_a3_hardware computeAdaptiveKd);
+                 per-joint zero_torque_kd_min/max below override the global values. -->
+            <param name="adaptive_kd_enabled">${adaptive_kd_enabled}</param>
+            <param name="zero_torque_kd">0.3</param>
+            <param name="zero_torque_kd_min">0.001</param>
+            <param name="zero_torque_kd_max">0.15</param>
+            <param name="kd_velocity_ref">1.0</param>
+            <param name="kd_smoothing_alpha">0.15</param>
           </xacro:if>
           <xacro:unless value="${use_real_hardware}">
@@ -41,12 +49,6 @@
           <!-- Gravity compensation feedforward parameters (100% gravity as feedforward torque, matching zero-torque mode) -->
           <param name="gravity_feedforward_ratio">1.0</param>  <!-- Gravity feedforward disabled -->
-          <!-- Zero-torque mode parameters -->
-          <param name="zero_torque_kd">0.3</param>  <!-- Fixed Kd fallback (used when adaptive_kd disabled) -->
-          <!-- Velocity-adaptive Kd parameters (Lorentzian decay + EMA smoothing) -->
-          <param name="adaptive_kd_enabled">true</param>
-          <param name="zero_torque_kd_min">0.001</param>  <!-- Kd at high speed (smooth feel) -->
-          <param name="zero_torque_kd_max">0.15</param>   <!-- Kd at rest (stability) -->
-          <param name="kd_velocity_ref">1.0</param>        <!-- Reference velocity where Kd drops to midpoint (rad/s) -->
-          <param name="kd_smoothing_alpha">0.15</param>    <!-- EMA smoothing factor (smaller = smoother transitions) -->
+          <!-- Adaptive-Kd params live in the real-hardware block above;
+               GenericSystem ignores them. -->
           <!-- Pinocchio dynamics model configuration -->
           <param name="urdf_path">$(find a3_description)/urdf/el_a3.urdf</param>

Commit message: Add F86: motor-side CAN timeout arming via 0x7028 (4000 counts=0.2s), vcan acceptance 29/29
Independent defense beyond the F81 host watchdog: on_activate writes the
uint32 timeout per motor (volatile, re-armed every enable), on_deactivate
disarms first. Host death is emulated with SIGKILL in the vcan acceptance;
all 7 motors self-reset at ~0.20 s. LL-089 records that 0x7028 is uint32
counts (~50us, 20000≈1s), correcting the old "float seconds" codec comment.

Co-Authored-By: Claude Sonnet 4.6 <noreply@anthropic.com>

File: src/a3_description/urdf/el_a3.urdf.xacro (robot description, xacro)
@@ -10,4 +10,6 @@
   <xacro:arg name="wrist_motor_type" default="EL05"/>
   <xacro:arg name="adaptive_kd_enabled" default="true"/>
+  <xacro:arg name="motor_can_timeout_enabled" default="true"/>
+  <xacro:arg name="motor_can_timeout_s" default="0.2"/>
   <!-- Wrist motor parameters (EL05: 6Nm, RS05: 5.5Nm) -->
   <xacro:property name="wrist_motor_type" value="$(arg wrist_motor_type)"/>
@@ -283,4 +285,6 @@
     host_can_id="$(arg host_can_id)"
     wrist_motor_type="$(arg wrist_motor_type)"
-    adaptive_kd_enabled="$(arg adaptive_kd_enabled)"/>
+    adaptive_kd_enabled="$(arg adaptive_kd_enabled)"
+    motor_can_timeout_enabled="$(arg motor_can_timeout_enabled)"
+    motor_can_timeout_s="$(arg motor_can_timeout_s)"/>
 </robot>

File: src/a3_description/urdf/el_a3_ros2_control.xacro (robot description, xacro)
@@ -2,5 +2,5 @@
 <!-- EL-A3 ros2_control configuration -->
 <robot xmlns:xacro="http://www.ros.org/wiki/xacro">
-  <xacro:macro name="el_a3_ros2_control" params="use_mock_hardware use_real_hardware can_interface host_can_id wrist_motor_type adaptive_kd_enabled">
+  <xacro:macro name="el_a3_ros2_control" params="use_mock_hardware use_real_hardware can_interface host_can_id wrist_motor_type adaptive_kd_enabled motor_can_timeout_enabled motor_can_timeout_s">
     <!-- Wrist motor effort limits based on motor type -->
     <xacro:property name="wrist_effort_max" value="${5.5 if wrist_motor_type == 'RS05' else 6.0}"/>
@@ -32,4 +32,9 @@
             <param name="kd_velocity_ref">1.0</param>
             <param name="kd_smoothing_alpha">0.15</param>
+            <!-- F86: arm motor-side CAN timeout (0x7028, uint32 counts ~50us, 20000≈1s).
+                 Independent of the F81 host watchdog: trips even if the host dies.
+                 0 / false disarms; firmware write is volatile, re-armed every on_activate. -->
+            <param name="motor_can_timeout_enabled">${motor_can_timeout_enabled}</param>
+            <param name="motor_can_timeout_s">${motor_can_timeout_s}</param>
           </xacro:if>
           <xacro:unless value="${use_real_hardware}">

Commit message: Add F98: L7 gripper limits synced to calibration [0.0,1.78], vcan acceptance 13/13
URDF joint limit, ros2_control position command_interface and MoveIt
joint_limits all carried the reBot reference +/-1.5708; the model
understated gripper travel by 12% and allowed physically meaningless
negative commands. L5/L6 genuine limits untouched. f87b regression 7/7.

Co-Authored-By: Claude Sonnet 4.6 <noreply@anthropic.com>

File: src/a3_description/urdf/el_a3.urdf.xacro (robot description, xacro)
@@ -255,5 +255,7 @@
     <child link="gripper_link"/>
     <axis xyz="0 0 1"/>
-    <limit effort="${wrist_effort}" velocity="50" lower="-1.5708" upper="1.5708"/>
+    <!-- F98: L7 calibrated 2026-09-13: open=0.0, mechanical stop 1.7825,
+         operational clamp 1.78; replaces reference ±1.5708. -->
+    <limit effort="${wrist_effort}" velocity="50" lower="0.0" upper="1.78"/>
     <dynamics damping="0.05" friction="0.05"/>
   </joint>

File: src/a3_description/urdf/el_a3_ros2_control.xacro (robot description, xacro)
@@ -270,7 +270,9 @@
         <param name="zero_torque_kd_min">0.02</param>
         <param name="zero_torque_kd_max">0.10</param>
-        <command_interface name="position">
-          <param name="min">-1.5708</param>
-          <param name="max">1.5708</param>
+        <!-- F98: position interface matches L7 calibration [0.0, 1.78]
+             (mechanical stop 1.7825); replaces reference ±1.5708. -->
+        <command_interface name="position">
+          <param name="min">0.0</param>
+          <param name="max">1.78</param>
         </command_interface>
         <command_interface name="velocity">

Commit message: F111-F123 补齐收口 + F124/F127 验收：named_poses 统一定义, servo_anchor/sim_push 薄桥, 零增益失能保活解耦, 0x18 周期下调; 修复 zero_to_ready 订阅匹配重试(logger 改 f-string 防 rclpy 多参 TypeError); 新增 f124/f126/f127 mock 验收脚本与 LL-130..138
Co-Authored-By: Claude Sonnet 4.6 <noreply@anthropic.com>

File: src/a3_description/urdf/el_a3.urdf.xacro (robot description, xacro)
@@ -12,4 +12,5 @@
   <xacro:arg name="motor_can_timeout_enabled" default="true"/>
   <xacro:arg name="motor_can_timeout_s" default="0.2"/>
+  <xacro:arg name="active_report_hz" default="10.0"/>
   <!-- Wrist motor parameters (EL05: 6Nm, RS05: 5.5Nm) -->
   <xacro:property name="wrist_motor_type" value="$(arg wrist_motor_type)"/>
@@ -289,4 +290,5 @@
     adaptive_kd_enabled="$(arg adaptive_kd_enabled)"
     motor_can_timeout_enabled="$(arg motor_can_timeout_enabled)"
-    motor_can_timeout_s="$(arg motor_can_timeout_s)"/>
+    motor_can_timeout_s="$(arg motor_can_timeout_s)"
+    active_report_hz="$(arg active_report_hz)"/>
 </robot>

File: src/a3_description/urdf/el_a3_ros2_control.xacro (robot description, xacro)
@@ -2,5 +2,5 @@
 <!-- EL-A3 ros2_control configuration -->
 <robot xmlns:xacro="http://www.ros.org/wiki/xacro">
-  <xacro:macro name="el_a3_ros2_control" params="use_mock_hardware use_real_hardware can_interface host_can_id wrist_motor_type adaptive_kd_enabled motor_can_timeout_enabled motor_can_timeout_s">
+  <xacro:macro name="el_a3_ros2_control" params="use_mock_hardware use_real_hardware can_interface host_can_id wrist_motor_type adaptive_kd_enabled motor_can_timeout_enabled motor_can_timeout_s active_report_hz">
     <!-- Wrist motor effort limits based on motor type -->
     <xacro:property name="wrist_effort_max" value="${5.5 if wrist_motor_type == 'RS05' else 6.0}"/>
@@ -37,4 +37,8 @@
             <param name="motor_can_timeout_enabled">${motor_can_timeout_enabled}</param>
             <param name="motor_can_timeout_s">${motor_can_timeout_s}</param>
+            <!-- F123: 0x18 active-report period (0x7026 EPScan_time), Hz.
+                 10 Hz → 100 ms → n=19 (factory default is 10 ms/100 Hz).
+                 Re-armed on every activate and after deactivate's reset. -->
+            <param name="active_report_hz">${active_report_hz}</param>
             <!-- F108: position-mode gravity feedforward (EDULITE
                  gravity_feedforward_ratio): t_ff = ratio * tau_scale * RNEA(q)
