Commit message: F168 native 6-joint product profile (drop L7 gripper); F169 a3_stack calibrate + F49 6J adaptation
F168: after the L7 gripper motor is removed (can1 has only motors 1..6),
the product stack previously had only a 7-joint profile -- the URDF
declared L7 and the hardware plugin aborted activation on 6/7 motors.
Add a native 6J profile that keeps MoveIt/JTC/melodion (unlike the F52
legacy-stack 5J fallback).

- el_a3.urdf.xacro: new include_gripper arg (default true); false omits
  L7_joint / gripper_link and passes through to the ros2_control macro
- el_a3_ros2_control.xacro: include_gripper param; false skips L7
- new el_a3_controllers_6j.yaml (no gripper_controller, zero_torque
  without L7), el_a3_6j.srdf (no gripper/arm_with_gripper group),
  motor_map_6j.yaml (power_sequence joints 1..6)
- a3_bringup.launch.py: include_gripper launch arg resolved in
  OpaqueFunction to select xacro/SRDF/controllers/fsm overrides/
  power_sequence map and skip the gripper spawner
- a3_stack.sh: probe accepts 7/7 or 1..6 (motor 7 missing) and
  auto-selects the profile; new --6j forces 6J; post-start /joint_states
  joint-count check. 7J remains the default and is unchanged.

F169: fold the gravity calibration scripts into a3_stack.sh calibrate
{model|scale} (preflight: stack running + READY + joint count, then
passes --joints 6|7 through), and make gravity_calibration.py (F49)
joint-count agnostic -- JOINT_NAMES/signs/pose lengths/tensor slices/
temperature checks all follow len() instead of a hardcoded 7. Default
--joints 7 behaviour is byte-for-byte unchanged.

Lessons: LL-157 (PythonExpression ternary concatenation precedence
swallowed include_gripper into the else branch; use OpaqueFunction for a
resolved boolean, verify with the three joints-count signals), LL-158
(F49's hardcoded 7 and the calibration entry-point consolidation).

Docs: QUICKSTART 6J section + calibrate usage, REQUIREMENTS index
F168/F169, scripts README.

File: src/a3_description/urdf/el_a3.urdf.xacro (robot description, xacro)
@@ -13,4 +13,8 @@
   <xacro:arg name="motor_can_timeout_s" default="0.2"/>
   <xacro:arg name="active_report_hz" default="10.0"/>
+  <!-- include_gripper：true=7 关节（L1–L7，含 L7 夹爪，默认）；
+       false=6 关节臂（拆掉 L7 夹爪电机）——不生成 L7_joint / gripper_link，
+       也不在 ros2_control 里声明 L7，配合 6J 档 SRDF/controllers 使用。 -->
+  <xacro:arg name="include_gripper" default="true"/>
   <!-- Wrist motor parameters (EL05: 6Nm, RS05: 5.5Nm) -->
   <xacro:property name="wrist_motor_type" value="$(arg wrist_motor_type)"/>
@@ -250,35 +254,39 @@
     <child link="end_effector"/>
   </joint>
-  <!-- Joint L7 (${wrist_motor_type} Motor 7 - Gripper, separate kinematic branch) -->
-  <joint name="L7_joint" type="revolute">
-    <origin xyz="0 0 -0.074" rpy="0 0 0"/>
-    <parent link="l5_l6_urdf_asm"/>
-    <child link="gripper_link"/>
-    <axis xyz="0 0 1"/>
-    <!-- F98: L7 calibrated 2026-09-13: open=0.0, mechanical stop 1.7825,
-         operational clamp 1.78; replaces reference ±1.5708. -->
-    <limit effort="${wrist_effort}" velocity="50" lower="0.0" upper="1.78"/>
-    <dynamics damping="0.05" friction="0.05"/>
-  </joint>
-  <link name="gripper_link">
-    <inertial>
-      <mass value="0.05"/>
-      <origin xyz="0 0 0"/>
-      <inertia ixx="0.0001" ixy="0" ixz="0" iyy="0.0001" iyz="0" izz="0.0001"/>
-    </inertial>
-    <visual>
-      <origin xyz="0 0 -0.0015" rpy="3.14159 0 0"/>
-      <geometry>
-        <mesh filename="package://a3_description/meshes/jaw.stl"/>
-      </geometry>
-      <material name="orange"/>
-    </visual>
-    <collision>
-      <origin xyz="0 0 -0.0015" rpy="3.14159 0 0"/>
-      <geometry>
-        <mesh filename="package://a3_description/meshes/jaw.stl"/>
-      </geometry>
-    </collision>
-  </link>
+  <!-- Joint L7 (${wrist_motor_type} Motor 7 - Gripper, separate kinematic branch)
+       include_gripper=false（6 关节臂）时不生成：L7 是独立分支（挂 l5_l6_urdf_asm），
+       去掉不影响 arm 组链（tip=end_effector）。 -->
+  <xacro:if value="$(arg include_gripper)">
+    <joint name="L7_joint" type="revolute">
+      <origin xyz="0 0 -0.074" rpy="0 0 0"/>
+      <parent link="l5_l6_urdf_asm"/>
+      <child link="gripper_link"/>
+      <axis xyz="0 0 1"/>
+      <!-- F98: L7 calibrated 2026-09-13: open=0.0, mechanical stop 1.7825,
+           operational clamp 1.78; replaces reference ±1.5708. -->
+      <limit effort="${wrist_effort}" velocity="50" lower="0.0" upper="1.78"/>
+      <dynamics damping="0.05" friction="0.05"/>
+    </joint>
+    <link name="gripper_link">
+      <inertial>
+        <mass value="0.05"/>
+        <origin xyz="0 0 0"/>
+        <inertia ixx="0.0001" ixy="0" ixz="0" iyy="0.0001" iyz="0" izz="0.0001"/>
+      </inertial>
+      <visual>
+        <origin xyz="0 0 -0.0015" rpy="3.14159 0 0"/>
+        <geometry>
+          <mesh filename="package://a3_description/meshes/jaw.stl"/>
+        </geometry>
+        <material name="orange"/>
+      </visual>
+      <collision>
+        <origin xyz="0 0 -0.0015" rpy="3.14159 0 0"/>
+        <geometry>
+          <mesh filename="package://a3_description/meshes/jaw.stl"/>
+        </geometry>
+      </collision>
+    </link>
+  </xacro:if>
   <!-- ros2_control interface -->
   <xacro:el_a3_ros2_control
@@ -291,4 +299,5 @@
     motor_can_timeout_enabled="$(arg motor_can_timeout_enabled)"
     motor_can_timeout_s="$(arg motor_can_timeout_s)"
-    active_report_hz="$(arg active_report_hz)"/>
+    active_report_hz="$(arg active_report_hz)"
+    include_gripper="$(arg include_gripper)"/>
 </robot>

File: src/a3_description/urdf/el_a3_ros2_control.xacro (robot description, xacro)
@@ -2,5 +2,5 @@
 <!-- EL-A3 ros2_control configuration -->
 <robot xmlns:xacro="http://www.ros.org/wiki/xacro">
-  <xacro:macro name="el_a3_ros2_control" params="use_mock_hardware use_real_hardware can_interface host_can_id wrist_motor_type adaptive_kd_enabled motor_can_timeout_enabled motor_can_timeout_s active_report_hz">
+  <xacro:macro name="el_a3_ros2_control" params="use_mock_hardware use_real_hardware can_interface host_can_id wrist_motor_type adaptive_kd_enabled motor_can_timeout_enabled motor_can_timeout_s active_report_hz include_gripper:=true">
     <!-- Wrist motor effort limits based on motor type -->
     <xacro:property name="wrist_effort_max" value="${5.5 if wrist_motor_type == 'RS05' else 6.0}"/>
@@ -346,4 +346,5 @@
         </xacro:if>
       </joint>
+      <xacro:if value="${include_gripper}">
       <!-- Joint L7 - ${wrist_motor_type} Motor 7 (Gripper) -->
       <joint name="L7_joint">
@@ -381,4 +382,5 @@
         </xacro:if>
       </joint>
+      </xacro:if>
     </ros2_control>
   </xacro:macro>
