Commit message: F174 default description -> 6-axis+linkage via a3_robot_model; de-hardcode description across bringup/sim chain
Introduce a3_robot_model, a system-level model config package: its
config/robot_model.yaml is the single source of truth for the default
description (package, xacro/static URDF, controllers, SRDF, motor_map,
joint_names, include_gripper), with field-level override from
~/.a3/robot_model.yaml. Default is now the 6-axis + linkage form
(a3_description_6j); pass --7j / include_gripper:=true to get the
7-axis gripper form.

Consumers now resolve through it instead of hardcoding a3_description:
a3_bringup.launch.py (OpaqueFunction builds from the resolved config;
never hardcodes package or profile file names), the sim chain
(edge_web_sim / edge_teleop_full_sim SRDF + URDF, which previously kept
the 7-axis SRDF and showed a gripper in RViz), sim_motor_node
(joint_names/tau_L7 no longer hardcoded -> no out-of-range on 6 joints),
a3_arm_controller/launch/arm_controller.launch.py (now injects
joint_names/switch_controllers/named_poses_pkg, fixing the F52 profile
mismatch), arm_controller (URDF path, description package, named-pose
pkg), gravity_torque_node, move_to_pose_ik_node, zero_to_ready_publisher
and the remaining bringup/moveit/cloud_edge launches. a3_stack.sh takes
its default profile from robot_model.yaml and adds --7j.

a3_description_6j: linkage now carries geometry/inertia instead of a
bare link -- a phi8 x 140mm cylinder placeholder (mass 0.02 kg, args
linkage_radius/length/mass) from the flange down to the TCP; the EL05
axis-6 housing stays (the motor is still present) while the L7 jaw mesh
is gone. Gripper-only configs (el_a3_controllers_6j.yaml,
gripper_*_plugin.yaml) are removed from the package, and the remaining
controllers/named_poses/rviz configs are cleaned for the gripper-free
form.

Lessons LL-163: switching the default description missed three hidden
hardcodes beyond a3_bringup.launch.py (sim launch SRDF + URDF,
sim_motor_node joint list, arm_controller launch without overrides) --
enumerate every entry that publishes the description or starts the
orchestration layer, and verify the three joint-count signals.

Docs: ROBOT_MODEL.md two-form section, REQUIREMENTS F174 ->
implemented-pending-hw, AGENT.md/CLAUDE.md checks and layering, docs
README package index, QUICKSTART.

File: src/a3_description_6j/urdf/el_a3.urdf (robot description, URDF)
Before this commit: robot EL-A3, 10 links, 9 joints
Links:
- link linkage_link: mass None -> 0.02; geometry collision cylinder length=0.14 radius=0.004; visual cylinder length=0.14 radius=0.004
Joints:
- joint linkage_joint: origin xyz=0 0 -0.014 rpy=0 0 0 -> xyz=0 0 -0.14 rpy=0 0 0

File: src/a3_description_6j/urdf/el_a3.urdf.xacro (robot description, xacro)
@@ -16,10 +16,24 @@
   <xacro:arg name="motor_can_timeout_s" default="0.2"/>
   <xacro:arg name="active_report_hz" default="10.0"/>
-  <!-- 连杆相对轴 6 的偏移（m）。-0.014 为初步估算，待实测后修正（F174）。 -->
-  <xacro:arg name="linkage_offset_z" default="-0.014"/>
+  <!-- 连杆相对轴 6 的偏移（m）。连杆从轴 6 法兰输出向下延伸，末端即 TCP；
+       长度按 14 cm 打印件估算，待实测/STP 到位后修正（F174）。 -->
+  <xacro:arg name="linkage_offset_z" default="-0.14"/>
+  <!-- 连杆圆柱占位参数（无 STP 前用圆柱代替）：
+       radius/length 单位 m，length = |linkage_offset_z|；mass 为打印件占位值（很轻），
+       换 STP 时只需替换下面的 cylinder 几何与 inertial。 -->
+  <xacro:arg name="linkage_radius" default="0.004"/>
+  <xacro:arg name="linkage_length" default="0.14"/>
+  <xacro:arg name="linkage_mass" default="0.02"/>
   <!-- Wrist motor parameters (EL05: 6Nm, RS05: 5.5Nm) -->
   <xacro:property name="wrist_motor_type" value="$(arg wrist_motor_type)"/>
   <xacro:property name="wrist_effort" value="${5.5 if wrist_motor_type == 'RS05' else 6.0}"/>
   <xacro:property name="linkage_offset_z" value="$(arg linkage_offset_z)"/>
+  <xacro:property name="linkage_radius" value="$(arg linkage_radius)"/>
+  <xacro:property name="linkage_length" value="$(arg linkage_length)"/>
+  <xacro:property name="linkage_mass" value="$(arg linkage_mass)"/>
+  <!-- 实心圆柱惯量（绕质心）：Izz = m·r²/2，Ixx = Iyy = m(3r²+L²)/12 -->
+  <xacro:property name="linkage_izz" value="${linkage_mass * linkage_radius * linkage_radius / 2.0}"/>
+  <xacro:property name="linkage_ixx"
+                  value="${linkage_mass * (3.0 * linkage_radius * linkage_radius + linkage_length * linkage_length) / 12.0}"/>
   <!-- Include ros2_control -->
   <xacro:include filename="$(find a3_description_6j)/urdf/el_a3_ros2_control.xacro"/>
@@ -170,5 +184,9 @@
     </collision>
   </link>
-  <!-- Link l5_l6_urdf_asm (轴 6 法兰输出) -->
+  <!-- Link l5_l6_urdf_asm (轴 6 法兰输出)
+       F174: 该 link 的视觉/碰撞为 el05_l6.stl（φ46×106mm 的 EL05 电机壳体，含输出轴段）——
+       对照实物（2026-10-15 确认）**这台电机仍在**，故整段保留（它同时占据连杆根部空间，
+       与连杆共轴：连杆圆柱 φ8 从法兰向下穿出）。原 7 轴形态里同处还有夹爪 jaw.stl（属已拆的
+       L7 输出），那部分已随 L7 一并去掉。 -->
   <link name="l5_l6_urdf_asm">
     <inertial>
@@ -178,5 +196,4 @@
                iyy="0.00177268" iyz="-7.87717e-06" izz="0.000610685"/>
     </inertial>
-    <!-- Part el05_l6 -->
     <visual>
       <origin xyz="0 0 -0.0755" rpy="3.14159 0 0"/>
@@ -248,9 +265,32 @@
     <dynamics damping="0.05" friction="0.05"/>
   </joint>
-  <!-- 连杆（6 轴形态的末端被动连杆，F174）
-       - 相对轴 6 法兰输出（l5_l6_urdf_asm）偏移 (0, 0, linkage_offset_z)，默认 -0.014 m（初步估算，待实测）
-       - 几何与惯量待实测：暂不给 visual/collision（RViz 不显示），也不写 <inertial>
-         （缺失 inertial 视为零质量，连杆暂不参与重力前馈模型），实测后补。 -->
-  <link name="linkage_link"/>
+  <!-- 连杆（6 轴形态的末端连杆，F174）
+       - 相对轴 6 法兰输出（l5_l6_urdf_asm）偏移 (0, 0, linkage_offset_z)，默认 -0.14 m
+         （14 cm 打印件；初步估算，待实测）
+       - 暂无 STP：用圆柱占位（radius/length/mass 见上方 xacro arg）。连杆本体在
+         linkage_link 是「法兰 → 末端（TCP）」这一段：linkage_link 原点落在末端，
+         所以圆柱形心在 +linkage_length/2 处，向上延伸到法兰。
+       - 质量 0.02 kg 为打印件占位值（很轻），参与重力前馈；换 STP 后一并修正。 -->
+  <link name="linkage_link">
+    <inertial>
+      <origin xyz="0 0 ${linkage_length / 2.0}" rpy="0 0 0"/>
+      <mass value="${linkage_mass}"/>
+      <inertia ixx="${linkage_ixx}" ixy="0" ixz="0"
+               iyy="${linkage_ixx}" iyz="0" izz="${linkage_izz}"/>
+    </inertial>
+    <visual>
+      <origin xyz="0 0 ${linkage_length / 2.0}" rpy="0 0 0"/>
+      <geometry>
+        <cylinder radius="${linkage_radius}" length="${linkage_length}"/>
+      </geometry>
+      <material name="orange"/>
+    </visual>
+    <collision>
+      <origin xyz="0 0 ${linkage_length / 2.0}" rpy="0 0 0"/>
+      <geometry>
+        <cylinder radius="${linkage_radius}" length="${linkage_length}"/>
+      </geometry>
+    </collision>
+  </link>
   <joint name="linkage_joint" type="fixed">
     <origin xyz="0 0 ${linkage_offset_z}" rpy="0 0 0"/>
@@ -258,6 +298,5 @@
     <child link="linkage_link"/>
   </joint>
-  <!-- End Effector link (TCP)：连杆末端。
-       连杆长度待实测，暂取连杆原点为 TCP（即 TCP 相对轴 6 = (0,0,-0.014)）。 -->
+  <!-- End Effector link (TCP)：连杆末端（linkage_link 原点即 TCP）。 -->
   <link name="end_effector"/>
   <joint name="end_effector_joint" type="fixed">

Commit message: F174 real CAD end piece (mm mesh, explicit placement) + SRDF collision entries + real-machine RViz preload
F174: the cylinder placeholder linkage_link is gone -- the end geometry is
now the real CAD STL el05_l6.stl attached directly to l5_l6_urdf_asm
(flange disc + phi46 section + phi10 rod, extending 150mm from the axis-6
flange; TCP at the rod end, linkage_tcp_z=-0.150). The mesh is exported
in millimetres with an off-link coordinate frame, so it is placed with
scale="0.001..." and explicit origin/rpy, all as xacro args
(linkage_mesh_scale/origin/rpy) so a re-export only changes those values.
jaw.stl removed; the old wrist housing mesh is archived (per the doc
comment) and the l5_l6_urdf_asm inertia keeps the calibrated wrist value.

el_a3_6j.srdf: the three linkage_link disable_collisions entries are no
longer needed (linkage_link removed); l5_l6_urdf_asm<->end_effector stays
Adjacent.

a3_bringup.launch.py: the real-machine entry point now preloads the
hide_randr shim like the sim entry (it previously only set
LIBGL_ALWAYS_SOFTWARE), fixing rviz2 dying immediately with exit -11 on
the real stack.

Lessons:
- LL-165: a new end-effector fixed part must be registered in the SRDF
  collision matrix, otherwise MoveIt sees an invalid self-collision start
  state and every move_group action fails with error 99999. Diagnosed
  with GetStateValidity (contacts name the pair and depth);
  disabling only the necessarily-overlapping pairs, restarting the stack
  after SRDF edits, and verifying via check_state_validity ->
  plan_kinematic_path.
- LL-166: measure a new STL's units and frame before wiring it into the
  URDF -- CAD parts are often mm with an assembly frame, so use scale +
  explicit origin/rpy, parameterise them, and re-check SRDF collisions
  after any part swap.
- LL-065 extended: both RViz entry points (sim and the unified real/
  sim product launch) must carry the hide_randr preload.

Docs: QUICKSTART 6-axis section, ROBOT_MODEL two-form section,
REQUIREMENTS F174 row, a3_description_6j README.

File: src/a3_description_6j/urdf/el_a3.urdf (robot description, URDF)
Before this commit: robot EL-A3, 10 links, 9 joints
Links:
- removed link linkage_link
- link l5_l6_urdf_asm: geometry collision mesh filename=package://a3_description_6j/meshes/el05_l6.stl scale=0.001 0.001 0.001; visual mesh filename=package://a3_description_6j/meshes/el05_l6.stl scale=0.001 0.001 0.001
Joints:
- removed joint linkage_joint
- joint end_effector_joint: origin xyz=0 0 0 rpy=0 0 0 -> xyz=0 0 -0.15 rpy=0 0 0; parent linkage_link -> l5_l6_urdf_asm

File: src/a3_description_6j/urdf/el_a3.urdf.xacro (robot description, xacro)
@@ -16,24 +16,22 @@
   <xacro:arg name="motor_can_timeout_s" default="0.2"/>
   <xacro:arg name="active_report_hz" default="10.0"/>
-  <!-- 连杆相对轴 6 的偏移（m）。连杆从轴 6 法兰输出向下延伸，末端即 TCP；
-       长度按 14 cm 打印件估算，待实测/STP 到位后修正（F174）。 -->
-  <xacro:arg name="linkage_offset_z" default="-0.14"/>
-  <!-- 连杆圆柱占位参数（无 STP 前用圆柱代替）：
-       radius/length 单位 m，length = |linkage_offset_z|；mass 为打印件占位值（很轻），
-       换 STP 时只需替换下面的 cylinder 几何与 inertial。 -->
-  <xacro:arg name="linkage_radius" default="0.004"/>
-  <xacro:arg name="linkage_length" default="0.14"/>
-  <xacro:arg name="linkage_mass" default="0.02"/>
+  <!-- 末端件（真实 STL，F174）：el05_l6.stl 由 CAD 导出，**单位 mm、坐标系与链接系不同**：
+       件自身轴线沿 mesh x，位于 mesh 的 (y,z) ≈ (0.5, 135.5) mm；贴合面 = mesh x = -42.15 mm 平面
+       （φ46 法兰盘那端），远端细杆端面 x = -192.15 mm → 件总长 150 mm。
+       下面 origin/scale 把它摆成「与轴 6 共轴、贴合面贴轴 6 法兰面 (link z = 0)、向末端伸出 150 mm」：
+         rpy = (0, -90°, 0)  → mesh +x 映射到 link +z（故 mesh 的 -x 方向 = 向末端）
+         xyz = (0.1355, -0.0005, 0.04215) m → 把 mesh 的轴线与贴合面搬到 link z 轴 / 原点
+       换件或重新导出 CAD 时只需改这两个值 + 下面的 TCP 偏移。 -->
+  <xacro:arg name="linkage_mesh_scale" default="0.001 0.001 0.001"/>
+  <xacro:arg name="linkage_mesh_origin" default="0.1355 -0.0005 0.04215"/>
+  <xacro:arg name="linkage_mesh_rpy" default="0 -1.5708 0"/>
+  <xacro:arg name="linkage_tcp_z" default="-0.150"/>
   <!-- Wrist motor parameters (EL05: 6Nm, RS05: 5.5Nm) -->
   <xacro:property name="wrist_motor_type" value="$(arg wrist_motor_type)"/>
   <xacro:property name="wrist_effort" value="${5.5 if wrist_motor_type == 'RS05' else 6.0}"/>
-  <xacro:property name="linkage_offset_z" value="$(arg linkage_offset_z)"/>
-  <xacro:property name="linkage_radius" value="$(arg linkage_radius)"/>
-  <xacro:property name="linkage_length" value="$(arg linkage_length)"/>
-  <xacro:property name="linkage_mass" value="$(arg linkage_mass)"/>
-  <!-- 实心圆柱惯量（绕质心）：Izz = m·r²/2，Ixx = Iyy = m(3r²+L²)/12 -->
-  <xacro:property name="linkage_izz" value="${linkage_mass * linkage_radius * linkage_radius / 2.0}"/>
-  <xacro:property name="linkage_ixx"
-                  value="${linkage_mass * (3.0 * linkage_radius * linkage_radius + linkage_length * linkage_length) / 12.0}"/>
+  <xacro:property name="linkage_mesh_scale" value="$(arg linkage_mesh_scale)"/>
+  <xacro:property name="linkage_mesh_origin" value="$(arg linkage_mesh_origin)"/>
+  <xacro:property name="linkage_mesh_rpy" value="$(arg linkage_mesh_rpy)"/>
+  <xacro:property name="linkage_tcp_z" value="$(arg linkage_tcp_z)"/>
   <!-- Include ros2_control -->
   <xacro:include filename="$(find a3_description_6j)/urdf/el_a3_ros2_control.xacro"/>
@@ -185,8 +183,7 @@
   </link>
   <!-- Link l5_l6_urdf_asm (轴 6 法兰输出)
-       F174: 该 link 的视觉/碰撞为 el05_l6.stl（φ46×106mm 的 EL05 电机壳体，含输出轴段）——
-       对照实物（2026-10-15 确认）**这台电机仍在**，故整段保留（它同时占据连杆根部空间，
-       与连杆共轴：连杆圆柱 φ8 从法兰向下穿出）。原 7 轴形态里同处还有夹爪 jaw.stl（属已拆的
-       L7 输出），那部分已随 L7 一并去掉。 -->
+       F174: 视觉/碰撞 = 真实末端件 el05_l6.stl（CAD 导出，mm 单位、外置坐标系，
+       见文件头 origin/scale 说明；旧电机壳网格留档为 meshes/el05_l6_bk.stl）。
+       惯量沿用腕部组件标定值（含末端件，标定即该形态实测）——换件后若质量差异明显再复核。 -->
   <link name="l5_l6_urdf_asm">
     <inertial>
@@ -197,14 +194,16 @@
     </inertial>
     <visual>
-      <origin xyz="0 0 -0.0755" rpy="3.14159 0 0"/>
-      <geometry>
-        <mesh filename="package://a3_description_6j/meshes/el05_l6.stl"/>
-      </geometry>
-      <material name="dark_brown"/>
-    </visual>
-    <collision>
-      <origin xyz="0 0 -0.0755" rpy="3.14159 0 0"/>
-      <geometry>
-        <mesh filename="package://a3_description_6j/meshes/el05_l6.stl"/>
+      <origin xyz="${linkage_mesh_origin}" rpy="${linkage_mesh_rpy}"/>
+      <geometry>
+        <mesh filename="package://a3_description_6j/meshes/el05_l6.stl"
+              scale="${linkage_mesh_scale}"/>
+      </geometry>
+      <material name="orange"/>
+    </visual>
+    <collision>
+      <origin xyz="${linkage_mesh_origin}" rpy="${linkage_mesh_rpy}"/>
+      <geometry>
+        <mesh filename="package://a3_description_6j/meshes/el05_l6.stl"
+              scale="${linkage_mesh_scale}"/>
       </geometry>
     </collision>
@@ -265,42 +264,11 @@
     <dynamics damping="0.05" friction="0.05"/>
   </joint>
-  <!-- 连杆（6 轴形态的末端连杆，F174）
-       - 相对轴 6 法兰输出（l5_l6_urdf_asm）偏移 (0, 0, linkage_offset_z)，默认 -0.14 m
-         （14 cm 打印件；初步估算，待实测）
-       - 暂无 STP：用圆柱占位（radius/length/mass 见上方 xacro arg）。连杆本体在
-         linkage_link 是「法兰 → 末端（TCP）」这一段：linkage_link 原点落在末端，
-         所以圆柱形心在 +linkage_length/2 处，向上延伸到法兰。
-       - 质量 0.02 kg 为打印件占位值（很轻），参与重力前馈；换 STP 后一并修正。 -->
-  <link name="linkage_link">
-    <inertial>
-      <origin xyz="0 0 ${linkage_length / 2.0}" rpy="0 0 0"/>
-      <mass value="${linkage_mass}"/>
-      <inertia ixx="${linkage_ixx}" ixy="0" ixz="0"
-               iyy="${linkage_ixx}" iyz="0" izz="${linkage_izz}"/>
-    </inertial>
-    <visual>
-      <origin xyz="0 0 ${linkage_length / 2.0}" rpy="0 0 0"/>
-      <geometry>
-        <cylinder radius="${linkage_radius}" length="${linkage_length}"/>
-      </geometry>
-      <material name="orange"/>
-    </visual>
-    <collision>
-      <origin xyz="0 0 ${linkage_length / 2.0}" rpy="0 0 0"/>
-      <geometry>
-        <cylinder radius="${linkage_radius}" length="${linkage_length}"/>
-      </geometry>
-    </collision>
-  </link>
-  <joint name="linkage_joint" type="fixed">
-    <origin xyz="0 0 ${linkage_offset_z}" rpy="0 0 0"/>
-    <parent link="l5_l6_urdf_asm"/>
-    <child link="linkage_link"/>
-  </joint>
-  <!-- End Effector link (TCP)：连杆末端（linkage_link 原点即 TCP）。 -->
+  <!-- End Effector link (TCP)：真实末端件（el05_l6.stl）的远端端面。
+       F174: 圆柱占位连杆 linkage_link 已删除——末端几何由上面 l5_l6_urdf_asm 的真实
+       STL 承担（该件从轴 6 法兰面伸出 150 mm，细杆端面即 TCP）。 -->
   <link name="end_effector"/>
   <joint name="end_effector_joint" type="fixed">
-    <origin xyz="0 0 0" rpy="0 0 0"/>
-    <parent link="linkage_link"/>
+    <origin xyz="0 0 ${linkage_tcp_z}" rpy="0 0 0"/>
+    <parent link="l5_l6_urdf_asm"/>
     <child link="end_effector"/>
   </joint>
